File: Kicad/Multimeter_Watch_Board_V1/Multimeter_Watch_Board_V1.kicad_pcb (KiCad board)
At the start: 2 copper layers, 17 parts, among them J1 AudioJack3_Ground_renamedPins, J2 AudioJack3_Ground_renamedPins, J3 AudioJack3_Ground_renamedPins, U1 PCF85163-SO08, Y1 32kHz

Commit message: start work on pcb layout
Parts:
- removed the R6 at (120.7, 49.5)
- removed the R6 at (128.3, 41.9)
- added BT1: Some Li-Po?, Connector_Molex:Molex_PicoBlade_53047-0210_1x02_P1.25mm_Vertical, F.Cu at (143.0, 59.0)
- added C1: 100n, Capacitor_SMD:C_0603_1608Metric_Pad1.05x0.95mm_HandSolder, F.Cu at (137.5, 130.5)
- added C2: 100n, Capacitor_SMD:C_0603_1608Metric_Pad1.05x0.95mm_HandSolder, F.Cu at (143.0, 51.0)
- added C3: 100n, Capacitor_SMD:C_0603_1608Metric_Pad1.05x0.95mm_HandSolder, F.Cu at (141.9, 130.5)
- added F1: Fuse, Fuse:Fuse_0805_2012Metric_Pad1.15x1.40mm_HandSolder, F.Cu at (112.8, 124.7)
- added J4: Conn_01x16_Female, Connector_PinSocket_2.54mm:PinSocket_1x16_P2.54mm_Vertical, F.Cu at (102.0, 53.0)
- added J5: Conn_01x16_Female, Connector_PinSocket_2.54mm:PinSocket_1x16_P2.54mm_Vertical, F.Cu at (153.0, 53.1)
- added R11: R, Resistor_SMD:R_0603_1608Metric_Pad1.05x0.95mm_HandSolder, F.Cu at (142.4, 102.2)
- added R12: R, Resistor_SMD:R_0603_1608Metric_Pad1.05x0.95mm_HandSolder, F.Cu at (137.7, 107.1)
- added R13: 1M, Resistor_SMD:R_0603_1608Metric_Pad1.05x0.95mm_HandSolder, F.Cu at (133.3, 109.6)
- added R14: 1M, Resistor_SMD:R_0603_1608Metric_Pad1.05x0.95mm_HandSolder, F.Cu at (117.0, 127.4)
- added R15: R, Resistor_SMD:R_2512_6332Metric_Pad1.52x3.35mm_HandSolder, F.Cu at (148.0, 54.0)
- added R16: 30, Resistor_SMD:R_2512_6332Metric_Pad1.52x3.35mm_HandSolder, F.Cu at (138.0, 54.0)
- added R6: R_shunt, Resistor_SMD:R_2512_6332Metric_Pad1.52x3.35mm_HandSolder, F.Cu at (125.0, 55.0)
- added U2: AD8592, Package_SO:MSOP-10_3x3mm_P0.5mm, F.Cu at (143.0, 54.0)
- moved R1 102.2 mm to (117.6, 121.8)
- moved R2 94.1 mm to (112.8, 121.8)
- moved R5 90.4 mm to (112.8, 118.8)
- moved R3 85.1 mm to (122.3, 118.6)
- moved R4 83.8 mm to (117.6, 118.8)
- moved U1 81.7 mm to (128.0, 67.0), turned to 180 degrees
- moved Y1 66.2 mm to (103.8, 134.3)
- moved J3 63.5 mm to (131.0, 55.0), turned to 270 degrees
- moved R7 61.5 mm to (112.6, 129.9)
- moved R8 58.4 mm to (117.4, 124.5)
- moved R9 57.5 mm to (112.6, 127.4)
- moved J1 53.4 mm to (108.0, 55.0), turned to 270 degrees
- moved R10 50.1 mm to (133.3, 107.1)
- moved CPU1 40.7 mm to (128.0, 80.0), turned to 180 degrees
- moved J2 8.79 mm to (118.0, 55.0), turned to 270 degrees
Connections:
- net Net-(CPU1-Pad17) renamed /AD11
- net Net-(CPU1-Pad20) renamed /AD10
- net Net-(R4-Pad2) renamed /ADC11
- CPU1 pad 10: Net-(CPU1-Pad10) -> /BUTT5
- CPU1 pad 11: Net-(CPU1-Pad11) -> /BUTT6
- CPU1 pad 12: Net-(CPU1-Pad12) -> /PB0
- CPU1 pad 13: Net-(CPU1-Pad13) -> /PB1
- CPU1 pad 14: Net-(CPU1-Pad14) -> /PB2
- CPU1 pad 15: Net-(CPU1-Pad15) -> /PB3
- CPU1 pad 16: Net-(CPU1-Pad16) -> /PB4
- CPU1 pad 18: Net-(CPU1-Pad18) -> /SWC
- CPU1 pad 19: Net-(CPU1-Pad19) -> /ADC6
- CPU1 pad 2: Net-(CPU1-Pad2) -> /PD4
- CPU1 pad 21: Net-(CPU1-Pad21) -> /SWD
- CPU1 pad 22: Net-(CPU1-Pad22) -> /ADC7
- CPU1 pad 23: Net-(CPU1-Pad23) -> /ADC0
- CPU1 pad 24: Net-(CPU1-Pad24) -> /ADC1
- CPU1 pad 25: Net-(CPU1-Pad25) -> /ADC2
- CPU1 pad 26: Net-(CPU1-Pad26) -> /ADC3
- CPU1 pad 27: Net-(CPU1-Pad27) -> /SCL
- CPU1 pad 28: Net-(CPU1-Pad28) -> /SDA
- CPU1 pad 29: Net-(CPU1-Pad29) -> /RESET
- CPU1 pad 3: Net-(CPU1-Pad3) -> /PE4
- CPU1 pad 30: Net-(CPU1-Pad30) -> /D0
- CPU1 pad 31: Net-(CPU1-Pad31) -> /D1
- CPU1 pad 4: Net-(CPU1-Pad4) -> /VCC
- CPU1 pad 5: Net-(CPU1-Pad5) -> /GND
- CPU1 pad 6: Net-(CPU1-Pad6) -> /BUTT1
- CPU1 pad 7: Net-(CPU1-Pad7) -> /BUTT2
- CPU1 pad 8: Net-(CPU1-Pad8) -> /BUTT3
- CPU1 pad 9: Net-(CPU1-Pad9) -> /BUTT4
- J2 pad 2: /ADC2 -> Net-(F1-Pad1)
- J3 pad 2: /A7 -> /ADC7
- J3 pad 3: /A6 -> /ADC6
- J3 pad 4: /DACout -> /ADC1
- R10 pad 1: /A7 -> /ADC7
- R2 pad 2: Net-(R2-Pad2) -> /PD3
- R3 pad 1: Net-(R2-Pad2) -> /PD3
- R3 pad 2: Net-(R3-Pad2) -> /PD2
- R4 pad 1: Net-(R3-Pad2) -> /PD2
- R7 pad 2: /A6 -> /ADC6
- R8 pad 2: /A6 -> /ADC6
- R9 pad 1: /A7 -> /ADC7
- U1 pad 4: Net-(U1-Pad4) -> /GND
- U1 pad 5: Net-(U1-Pad5) -> /SDA
- U1 pad 6: Net-(U1-Pad6) -> /SCL
- U1 pad 8: Net-(U1-Pad8) -> /VCC
- Y1 pad 1: Net-(Y1-Pad1) -> Net-(U1-Pad2)
- Y1 pad 2: Net-(Y1-Pad2) -> Net-(U1-Pad1)
Other:
- board outline added: 55 x 45 mm
- copper layers 2 -> 4

Commit message: Switch left and right pin headers (for simpler DACout and VCChalf routing)
Parts:
- moved J4 51.0 mm to (153.0, 53.0)
- moved J5 51.0 mm to (102.0, 53.1)
Changed lines of the file:
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@@
   )
   (module Connector_PinSocket_2.54mm:PinSocket_1x16_P2.54mm_Vertical (layer F.Cu)
-    (at 153 53.06)
+    (at 102 53.06)
     (descr "Through hole straight socket strip, 1x16, 2.54mm pitch, single row (from Kicad 4.0.7), script generated")
     (tags "Through hole socket strip THT 1x16 2.54mm single row")
@@
   )
   (module Connector_PinSocket_2.54mm:PinSocket_1x16_P2.54mm_Vertical (layer F.Cu)
-    (at 102 53)
+    (at 153 53)
     (descr "Through hole straight socket strip, 1x16, 2.54mm pitch, single row (from Kicad 4.0.7), script generated")
     (tags "Through hole socket strip THT 1x16 2.54mm single row")

Commit message: first attempt at processor board layout
Parts:
- U1: footprint Package_SO:SOIC-8-1EP_3.9x4.9mm_P1.27mm_EP2.29x3mm -> Package_SO:SOIC-8-N7_3.9x4.9mm_P1.27mm
- moved R14 75.0 mm to (147.6, 59.0), turned to 180 degrees
- moved F1 66.4 mm to (125.5, 59.5)
- moved R9 63.8 mm to (127.9, 65.5), turned to 180 degrees
- moved R7 62.3 mm to (127.9, 69.5)
- moved R8 57.9 mm to (127.9, 67.5)
- moved C3 57.8 mm to (136.0, 73.0), turned to 135 degrees
- moved Y1 55.8 mm to (137.0, 89.5), turned to 270 degrees
- moved R13 51.1 mm to (147.6, 60.5)
- moved R5 47.2 mm to (106.5, 72.0), turned to 115 degrees
- moved C1 46.8 mm to (142.6, 84.0)
- moved R10 43.9 mm to (127.9, 63.5), turned to 180 degrees
- moved R4 43.8 mm to (109.2, 75.8), turned to 140 degrees
- moved R2 41.8 mm to (118.0, 80.2), turned to 165 degrees
- moved R1 41.0 mm to (122.5, 81.0), turned to 180 degrees
- moved R3 41.0 mm to (113.6, 78.6), turned to 155 degrees
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Connections:
- CPU1 pad 17: /AD11 -> /ADC11
- CPU1 pad 20: /AD10 -> /ADC10
- F1 pad 2: /ADC2 -> /ADC3
- J2 pad 2: Net-(F1-Pad1) -> /ADC2
- J2 pad 3: /ADC3 -> Net-(F1-Pad1)
- J4 pad 1: /SCL -> /VCC
- J4 pad 10: /VCC_HALF -> /SDA
- J4 pad 11: /SWC -> /SCL
- J4 pad 13: /RESET -> /SWC
- J4 pad 15: /PE4 -> /SDA
- J4 pad 16: /VCC -> /SCL
- J4 pad 2: /BUTT1 -> /BUTT2
- J4 pad 3: /BUTT2 -> /BUTT1
- J4 pad 4: /TODO_GND -> /GND
- J4 pad 5: /ADC7 -> /VCC_HALF
- J4 pad 6: /ADC6 -> /ADC1
- J4 pad 7: /ADC1 -> /RESET
- J4 pad 8: /SCL -> /ADC6
- J4 pad 9: /SDA -> /ADC7
- J5 pad 1: /SDA -> /GND
- J5 pad 16: /GND -> /PE4
- R1 pad 2: Net-(R1-Pad2) -> /ADC10
- R2 pad 1: Net-(R1-Pad2) -> /ADC10
Routing:
- net /PE4: track 0.00 -> 87.0 mm, vias 0 -> 4
- net /ADC1: track 0.00 -> 68.9 mm, vias 0 -> 2
- net Net-(J1-Pad2): track 0.00 -> 64.7 mm, vias 0 -> 2
- net /ADC7: track 0.00 -> 63.9 mm, vias 0 -> 4
- net /ADC6: track 0.00 -> 62.2 mm, vias 0 -> 3
- net /ADC0: track 0.00 -> 58.4 mm, vias 0 -> 2
- net /SDA: track 0.00 -> 55.0 mm
- net /SWC: track 0.00 -> 53.8 mm
- net /SCL: track 0.00 -> 48.1 mm
- net /D1: track 0.00 -> 44.3 mm, vias 0 -> 2
- net /D0: track 0.00 -> 42.6 mm, vias 0 -> 2
- net /ADC2: track 0.00 -> 40.3 mm, vias 0 -> 2
- net /PD2: track 0.00 -> 40.2 mm, vias 0 -> 2
- net /VCC: track 0.00 -> 37.7 mm, vias 0 -> 4
- net /ADC3: track 0.00 -> 36.4 mm, vias 0 -> 2
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- added copper zone on In1.Cu, net /GND
- added copper zone on In2.Cu, net /VCC
