File: Kicad/Multimeter_Watch_Board_V1/Multimeter_Watch_Board_V1.sch (KiCad schematic (older format))
At the start: 34 parts, among them J1 AudioJack3_Ground_renamedPins, J2 AudioJack3_Ground_renamedPins, J3 AudioJack3_Ground_renamedPins, J4 Conn_01x16_Female, J5 Conn_01x16_Female, U1 PCF85163-SO08, U2 AD8592, Y1 32kHz

Commit message: display board done, todo: move display down to allow for jack labels
Connections:
- net SCL: now also J4.10 (Pin_10), R11.2; no longer J4.11 (Pin_11), R12.2
- net SDA: now also J4.11 (Pin_11), R12.2; no longer J4.10 (Pin_10), R11.2
Other:
- moved on the sheet: R11, R12
Changed lines of the file:
@@
 L Device:R R11
 U 1 1 5F234AFA
+P 5750 4800
+F 0 "R11" H 5820 4846 50  0000 L CNN
+F 1 "R" H 5820 4755 50  0000 L CNN
+F 2 "Resistor_SMD:R_0603_1608Metric_Pad1.05x0.95mm_HandSolder" V 5680 4800 50  0001 C CNN
+F 3 "~" H 5750 4800 50  0001 C CNN
+	1    5750 4800
+	1    0    0    -1
+$EndComp
+$Comp
+L Device:R R12
+U 1 1 5F2353C3
 P 6050 4800
-F 0 "R11" H 6120 4846 50  0000 L CNN
+F 0 "R12" H 6120 4846 50  0000 L CNN
 F 1 "R" H 6120 4755 50  0000 L CNN
 F 2 "Resistor_SMD:R_0603_1608Metric_Pad1.05x0.95mm_HandSolder" V 5980 4800 50  0001 C CNN
 F 3 "~" H 6050 4800 50  0001 C CNN
 	1    6050 4800
-	1    0    0    -1
-$EndComp
-$Comp
-L Device:R R12
-U 1 1 5F2353C3
-P 5750 4800
-F 0 "R12" H 5820 4846 50  0000 L CNN
-F 1 "R" H 5820 4755 50  0000 L CNN
-F 2 "Resistor_SMD:R_0603_1608Metric_Pad1.05x0.95mm_HandSolder" V 5680 4800 50  0001 C CNN
-F 3 "~" H 5750 4800 50  0001 C CNN
-	1    5750 4800
 	1    0    0    -1
 $EndComp
@@
 Text Label 9800 4800 0    50   ~ 0
 GND
+Text Label 9800 5400 0    50   ~ 0
+SCL
 Text Label 9800 5500 0    50   ~ 0
-SCL
-Text Label 9800 5400 0    50   ~ 0
 SDA
 Wire Wire Line
