File: Kicad/Multimeter_Watch_DisplayBoard_V1/Multimeter_Watch_DisplayBoard_V1.kicad_pcb (KiCad board)
At the start: 2 copper layers, 55 x 46 mm, 32 parts, among them J1 Conn_01x03_Male, J2 Conn_01x03_Male, J3 Conn_01x03_Male, J4 Conn_01x03_Male, Q1 A03400A N-MOS, SW1 SW_Push, SW2 SW_Push, SW3 SW_Push, SW4 SW_Push, SW5 SW_Push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

Commit message: replace temp holes with actual drill holes
Parts:
- added Hole1: MountingHole_2.1mm, MountingHole:MountingHole_2.1mm, B.Cu at (119.7, 84.5)
- added Hole2: MountingHole_2.1mm, MountingHole:MountingHole_2.1mm, B.Cu at (143.3, 84.5)
Routing:
- net /SDA: track 45.6 -> 47.7 mm
- net /GND: vias 13 -> 16
- net /BUTT4: vias 1 -> 0
Other:
- outline, holes or cut-outs redrawn
- board text added: "Temporary edge cuts replaced with actual holes"
- board text removed: "TEMPORARY todo:replace with actual drill holes"

Commit message: group rlc tester pins on right header
Parts:
- removed J_placeholder2: Conn_01x16_Female, Connector_PinSocket_2.54mm:PinSocket_1x16_P2.54mm_Vertical

Commit message: Refactor button handling and adjust button pinout for compatibility with the new hardware. Implement sleep + wakeup; implement r/w to RTC chip. Fix clock to correctly read the actual value from the RTC. Implement setting of the current time. Implement a hotkey-based menu. Implement a 6-key keyboard proof of concept. Add utility functions for adc/pga reading. Implement a basic linear cc/cv power supply.Implement a function generator proof-of concept. Minor changes and refactoring.
Parts:
- removed J_placeholder1: Conn_01x16_Female, Connector_PinSocket_2.54mm:PinSocket_1x16_P2.54mm_Vertical
