File: Kicad/V2/Multimeter_Watch_DisplayBoard/Multimeter_Watch_DisplayBoard.kicad_pcb (KiCad board)
At the start: 2 copper layers, 46 x 42 mm, 15 parts, among them J1 51281-1294, SW1 SW_Push, SW2 SW_Push, SW3 SW_Push, SW4 SW_Push, SW5 SW_Push, SW6 SW_Push

Commit message: drc update for displayboard
Other:
- net class Default: clearance 0.2 -> 0.15
- rule trace_clearance: 0.2 -> 0.15
- rule trace_min: 0.2 -> 0.15
